Commit message: fix issue in cartpole.urdf from previous commit

File: common/test/urdf/cartpole_robot/cartpole.urdf (robot description, URDF)
Before this commit: robot cartpole_robot, 3 links, 2 joints
Links:
- link rail: mass 100.0 -> None

Commit message: add plugin for cartpole

File: common/test/urdf/cartpole_robot/cartpole.urdf (robot description, URDF)
Before this commit: robot cartpole_robot, 3 links, 2 joints
Links:
- link cart: mass None -> 1
- link pole: mass None -> 1
- link rail: mass None -> 0
Joints:
- joint slider_cart: limit lower=-0.42 upper=0.42 effort=1 velocity=20 -> lower=-0.42 upper=0.42 effort=1000 velocity=20
